File: retr3d-testbench.sch (EAGLE design)
At the start: 72 parts, among them U1 ARDUINO-MEGAFULL

Commit message: Added SMD one sided version
Parts:
- GND, LED, RA0, RA1, RA10, RA11, RA12, RA13, RA14, RA15, RA2, RA3, RA4, RA5, RA6, RA7, RA8, RA9, RD10, RD11, RD12, RD13, RD14, RD15, RD16, RD17, RD18, RD19, RD2, RD20, RD21, RD22, RD23, RD24, RD25, RD26, RD28, RD29, RD3, RD30, RD31, RD32, RD33, RD34, RD35, RD36, RD37, RD38, RD39, RD4, RD40, RD41, RD42, RD43, RD44, RD45, RD46, RD47, RD48, RD49, RD5, RD50, RD51, RD52, RD53, RD6, RD7, RD8, RD9, VCC: device eagle-ltspice:R0207/10 -> SparkFun-Resistors:RESISTOR0805-RES
- LED1: device led:LED5MM -> masterperson40:LEDRETR3D
- U1: value ARDUINO-MEGAFULL -> ARDUINO-MEGAARDUINO_MEGA_MINIMAL; device SparkFun-Boards:ARDUINO-MEGAFULL -> masterperson40:ARDUINO-MEGAARDUINO_MEGA_MINIMAL
Connections:
- new net N$6: LED1.C, U1.GND@4
- net GND: now also U1.GND@1; no longer LED1.C, U1.GND@4
